Commit message: adapted urdf for tests on bot

File: urdf/camera.urdf.xacro (robot description, xacro)
@@ -14,5 +14,5 @@
     <joint name="cam_stereo_joint" type="fixed">
         <origin xyz="0.07 0.06 0.08" rpy="0 0 0"/>
-        <parent link="chassis"/>
+        <parent link="base_link"/>
         <child link="cam_stereo"/>
     </joint>

File: urdf/chassis.urdf.xacro (robot description, xacro)
@@ -5,5 +5,5 @@
     <xacro:property name="chassis_width" value=".19"/>
     <xacro:property name="chassis_height" value="0.070"/>
-    <link name="chassis">
+    <link name="base_link">
         <visual>
             <origin rpy="-${PI/2} 0 ${PI/2}" xyz="0 0 0"/>

File: urdf/sonar.urdf.xacro (robot description, xacro)
@@ -13,5 +13,5 @@
     <joint name="sonar_front_joint" type="fixed">
         <origin xyz="0.07 0 0.08" rpy="0 0 0"/>
-        <parent link="chassis"/>
+        <parent link="base_link"/>
         <child link="sonar_front"/>
     </joint>

File: urdf/wheels.urdf.xacro (robot description, xacro)
@@ -19,5 +19,5 @@
     <xacro:macro name="wheel" params= "prefix suffix X Y Z">
       <link name= "${prefix}_${suffix}_wheel">
-        <visual>
+       <visual>
          <origin rpy= "${PI/2} 0 0" xyz= "0 0 0"/>
          <geometry><cylinder length="${wheel_width}" radius= "${wheel_radius/5}"/></geometry>
@@ -48,5 +48,5 @@
       </joint>
     <joint name="${prefix}_${suffix}_wheel_joint" type="continuous">
-      <parent link= "chassis"/>
+      <parent link= "base_link"/>
       <child link= "${prefix}_${suffix}_wheel"/>
       <origin xyz= "${0.062*X-0.058*Y} ${(chassis_len/2+0.02)*Z}  0.015" rpy="0 0 0"/>
@@ -66,7 +66,7 @@
      </transmission>
     </xacro:macro>
-    <xacro:wheel prefix="right" suffix="front" X="1" Y="0" Z="-1"/>
-    <xacro:wheel prefix="right" suffix="back" X="0" Y="1" Z="-1"/>
-    <xacro:wheel prefix="left" suffix="front" X="1" Y="0" Z="1"/>
-    <xacro:wheel prefix="left" suffix="back" X="0" Y="1" Z="1"/>
+    <xacro:wheel prefix="right" suffix="" X="0" Y="1" Z="-1"/>
+    <xacro:wheel prefix="left" suffix="" X="0" Y="1" Z="1"/>
+   <!-- <xacro:wheel prefix="right" suffix="front" X="1" Y="1" Z="-1"/>
+     <xacro:wheel prefix="left" suffix="front" X="1" Y="1" Z="1"/>-->
 </robot>
