Commit message: renamed

File: urdf/chassis.urdf.xacro (robot description, xacro)
@@ -9,5 +9,5 @@
             <origin rpy="-${PI/2} 0 ${PI/2}" xyz="0 0 0"/>
             <geometry>
-                <mesh filename="package://robopi/meshes/base assembly.dae"/>
+                <mesh filename="package://robopi/meshes/base_assembly.dae"/>
             </geometry>
         </visual>
@@ -15,5 +15,5 @@
             <origin rpy="-${PI/2} 0 0" xyz="0 0 0"/>
             <geometry>
-                <mesh filename="package://robopi/meshes/base assembly.dae"/>
+                <mesh filename="package://robopi/meshes/base_assembly.dae"/>
             </geometry>
         </collision>
